Commit message: Modify side camera positions to output a lateral FOV

File: parc_robot_description/urdf/side_cameras.xacro (robot description, xacro)
@@ -14,4 +14,5 @@
       </inertial>
       <visual>
+        <origin xyz="0.0 0.015 0.0" rpy="0 -${pi/2} 0"/>
         <geometry>
           <mesh filename="package://parc_robot_description/meshes/ZED2.dae"/>
@@ -19,4 +20,5 @@
       </visual>
       <collision>
+        <origin xyz="0.0 0.015 0.0" rpy="0 0 0"/>
         <geometry>
           <mesh filename="package://parc_robot_description/meshes/ZED2.dae"/>
@@ -88,4 +90,5 @@
       </inertial>
       <visual>
+        <origin xyz="0.0 0.015 0.0" rpy="0 ${pi/2} 0"/>
         <geometry>
           <mesh filename="package://parc_robot_description/meshes/ZED2.dae"/>
@@ -93,4 +96,5 @@
       </visual>
       <collision>
+        <origin xyz="0.0 0.015 0.0" rpy="0 0 0"/>
         <geometry>
           <mesh filename="package://parc_robot_description/meshes/ZED2.dae"/>
