Commit message: Implement ros2_control on PARC robot

File: parc_robot_description/urdf/parc_robot.xacro (robot description, xacro)
@@ -1,5 +1,4 @@
 <?xml version="1.0"?>
 <robot name="parc_robot_v2" xmlns:xacro="http://ros.org/wiki/xacro">
-  <!-- <xacro:include filename="$(find parc_robot_description)/urdf/parc_robot_v2.xacro" /> -->
   <xacro:arg name="robot_namespace" default="/" />
   <xacro:arg name="urdf_extras" default="empty.urdf" />

File: parc_robot_description/urdf/parc_robot_gazebo.xacro (robot description, xacro)
@@ -1,35 +1,41 @@
 <?xml version="1.0"?>
-<!--
-Reference:
-    [1] https://answers.ros.org/question/246914/four-wheeled-skid-steering-in-gazebo-and-ros-using-gazebo-ros-control/
-    [2] https://answers.ros.org/question/10119/gazebo-controller-for-skid-steering/
-    [3] https://answers.ros.org/question/9640/rotation-error-in-gazebo-simulation/
-    [4] https://www.youtube.com/watch?v=fuRAv6PDwdw
--->
 <robot xmlns:xacro="http://ros.org/wiki/xacro">
-  <xacro:include filename="$(find parc_robot_description)/urdf/scout_wheel.gazebo" />
-  <!-- Additional definitions for simulation -->
-  <!-- <gazebo reference="base_link">
-      <material>Gazebo/Grey</material>
-  </gazebo> -->
-  <!-- Actuator configurations -->
-  <xacro:scout_wheel_transmission wheel_prefix="front_right" />
-  <xacro:scout_wheel_transmission wheel_prefix="front_left" />
-  <xacro:scout_wheel_transmission wheel_prefix="rear_left" />
-  <xacro:scout_wheel_transmission wheel_prefix="rear_right" />
-  <!-- Controller configurations -->
-  <gazebo>
-    <plugin name="gazebo_ros_control" filename="libgazebo_ros_control.so">
-			<robotNamespace>/</robotNamespace>
-			<!-- <robotSimType>steer_bot_hardware_gazebo/SteerBotHardwareGazebo</robotSimType> -->
-      <robotSimType>gazebo_ros_control/DefaultRobotHWSim</robotSimType>
-    </plugin>
-  </gazebo>
-	<!-- <gazebo>
-    <plugin name="joint_state_publisher" filename="libgazebo_ros_joint_state_publisher.so">
-      <jointName>front_left_wheel, front_right_wheel, rear_left_wheel, rear_right_wheel</jointName>
-    </plugin>
-  </gazebo> -->
-  <!-- kp spring constant, kd damping constant -->
+  <ros2_control name='GazeboSystem' type='system'>
+    <hardware>
+      <plugin>gazebo_ros2_control/GazeboSystem</plugin>
+    </hardware>
+    <joint name='front_left_wheel'>
+      <command_interface name='velocity'>
+        <param name='min'>-10</param>
+        <param name='max'>10</param>
+      </command_interface>
+      <state_interface name='velocity'/>
+      <state_interface name='position'/>
+    </joint>
+    <joint name='front_right_wheel'>
+      <command_interface name='velocity'>
+        <param name='min'>-10</param>
+        <param name='max'>10</param>
+      </command_interface>
+      <state_interface name='velocity'/>
+      <state_interface name='position'/>
+    </joint>
+    <joint name='rear_left_wheel'>
+      <command_interface name='velocity'>
+        <param name='min'>-10</param>
+        <param name='max'>10</param>
+      </command_interface>
+      <state_interface name='velocity'/>
+      <state_interface name='position'/>
+    </joint>
+    <joint name='rear_right_wheel'>
+      <command_interface name='velocity'>
+        <param name='min'>-10</param>
+        <param name='max'>10</param>
+      </command_interface>
+      <state_interface name='velocity'/>
+      <state_interface name='position'/>
+    </joint>
+  </ros2_control>
   <gazebo>
     <mu1 value="1.0"/>
@@ -42,32 +48,8 @@
   </gazebo>
   <gazebo>
-    <plugin name="skid_steer_drive_controller" filename="libgazebo_ros_skid_steer_drive.so">
-      <updateRate>100.0</updateRate>
-      <robotNamespace>/</robotNamespace>
-      <leftFrontJoint>front_left_wheel</leftFrontJoint>
-      <rightFrontJoint>front_right_wheel</rightFrontJoint>
-      <leftRearJoint>rear_left_wheel</leftRearJoint>
-      <rightRearJoint>rear_right_wheel</rightRearJoint>
-      <wheelSeparation>4</wheelSeparation>
-      <wheelDiameter>0.32918</wheelDiameter>
-      <robotBaseFrame>base_link</robotBaseFrame>
-      <torque>1000</torque>
-      <commandTopic>cmd_vel</commandTopic>
-      <broadcastTF>true</broadcastTF>
-      <odometryTopic>odom</odometryTopic>
-      <odometryFrame>odom</odometryFrame>
-      <covariance_x>0.000100</covariance_x>
-      <covariance_y>0.000100</covariance_y>
-      <covariance_yaw>0.010000</covariance_yaw>
+    <plugin name='gazebo_ros2_control' filename='libgazebo_ros2_control.so'>
+      <parameters>$(find parc_robot_bringup)/config/controllers.yaml</parameters>
+      <parameters>$(find parc_robot_bringup)/config/gazebo_ros2_ctl_use_sim.yaml</parameters>
     </plugin>
   </gazebo>
-  <!-- <gazebo>
-    <plugin name="object_controller" filename="libgazebo_ros_planar_move.so">
-      <commandTopic>cmd_vel</commandTopic>
-      <odometryTopic>odom</odometryTopic>
-      <odometryFrame>odom</odometryFrame>
-      <odometryRate>20.0</odometryRate>
-      <robotBaseFrame>base_footprint</robotBaseFrame>
-    </plugin>
-  </gazebo> -->
 </robot>

File: parc_robot_description/urdf/sensors.xacro (robot description, xacro)
@@ -9,5 +9,4 @@
   <xacro:ydlidar_sensor parent="base_link">
     <origin xyz="0.25 0 0.18" rpy="0 0 0" />
-    <!-- <origin xyz="0.25 0 0.14" rpy="0 0 0" /> -->
   </xacro:ydlidar_sensor>
   <!-- zed2 camera -->
@@ -22,10 +21,8 @@
   <xacro:left_side_camera parent="base_link">
     <origin xyz="0 0.55 0.635" rpy="0 1.5708 1.571428571"/>
-    <!-- <origin xyz="0 0.7 0.7" rpy="0 1.0472 1.571428571"/> -->
   </xacro:left_side_camera>
     <!-- right_side_camera -->
   <xacro:right_side_camera parent="base_link">
     <origin xyz="0 -0.55 0.635" rpy="0 1.5708 1.571428571"/>
-    <!-- <origin xyz="0 -0.7 0.7" rpy="0 2.0944 1.571428571"/> -->
   </xacro:right_side_camera>
 </robot>

File: parc_robot_description/urdf/side_cameras.xacro (robot description, xacro)
@@ -63,5 +63,5 @@
           </distortion>
         </camera>
-        <plugin name="camera_controller" filename="libgazebo_ros_camera.so">
+        <plugin name="left_camera_controller" filename="libgazebo_ros_camera.so">
           <!-- <robotNamespace>${robot_ns}</robotNamespace> -->
           <cameraName>left_camera</cameraName>
@@ -139,5 +139,5 @@
           </distortion>
         </camera>
-        <plugin name="camera_controller" filename="libgazebo_ros_camera.so">
+        <plugin name="right_camera_controller" filename="libgazebo_ros_camera.so">
           <!-- <robotNamespace>${robot_ns}</robotNamespace> -->
           <cameraName>right_camera</cameraName>

File: parc_robot_description/urdf/zed2.xacro (robot description, xacro)
@@ -81,11 +81,4 @@
     </joint>
     <link name="zed2_temp_right_link" />
-  <!-- </xacro:macro> -->
-  <!-- <xacro:macro name="zed2_gazebo"> -->
-  <!-- <xacro:macro name="zed2_gazebo" params="robot_ns:=''"> -->
-    <!-- <xacro:property name="link_prefix" value=""/>
-    <xacro:if value="${robot_ns != '' and robot_ns != '/'}">
-      <xacro:property name="link_prefix" value="${robot_ns}/"/>
-    </xacro:if> -->
     <gazebo reference="zed2_camera_center">
       <sensor type="camera" name="zed2_center_camera">
@@ -118,6 +111,5 @@
           </distortion>
         </camera>
-        <plugin name="camera_controller" filename="libgazebo_ros_camera.so">
-          <!-- <robotNamespace>${robot_ns}</robotNamespace> -->
+        <plugin name="zed2_center_camera_controller" filename="libgazebo_ros_camera.so">
           <cameraName>camera</cameraName>
           <imageTopicName>image_raw</imageTopicName>
@@ -165,6 +157,5 @@
           </distortion>
         </camera>
-        <plugin name="camera_controller" filename="libgazebo_ros_camera.so">
-          <!-- <robotNamespace>${robot_ns}</robotNamespace> -->
+        <plugin name="zed2_left_camera_controller" filename="libgazebo_ros_camera.so">
           <cameraName>zed2/left_raw</cameraName>
           <imageTopicName>image_raw_color</imageTopicName>
@@ -182,5 +173,5 @@
         </plugin>
       </sensor>
-      <sensor type="depth" name="zed2_left_camera">
+      <sensor type="depth" name="zed2_leftd_camera">
         <!-- Rectified images, Depth images, Point Clouds -->
         <always_on>true</always_on>
@@ -204,6 +195,5 @@
           </noise>
         </camera>
-        <plugin name="camera_controller" filename="libgazebo_ros_openni_kinect.so">
-          <!-- <robotNamespace>${robot_ns}</robotNamespace> -->
+        <plugin name="zed2_leftd_camera_controller" filename="libgazebo_ros_openni_kinect.so">
           <cameraName>zed2</cameraName>
           <imageTopicName>left/image_rect_color</imageTopicName>
@@ -255,6 +245,5 @@
           </distortion>
         </camera>
-        <plugin name="camera_controller" filename="libgazebo_ros_camera.so">
-          <!-- <robotNamespace>${robot_ns}</robotNamespace> -->
+        <plugin name="zed2_right_camera_controller" filename="libgazebo_ros_camera.so">
           <cameraName>zed2/right_raw</cameraName>
           <imageTopicName>image_raw_color</imageTopicName>
@@ -294,6 +283,5 @@
           </noise>
         </camera>
-        <plugin name="camera_controller" filename="libgazebo_ros_camera.so">
-          <!-- <robotNamespace>${robot_ns}</robotNamespace> -->
+        <plugin name="zed2_rightrect_camera_controller" filename="libgazebo_ros_camera.so">
           <cameraName>zed2/right</cameraName>
           <imageTopicName>image_rect_color</imageTopicName>
@@ -312,5 +300,4 @@
         <update_rate>100</update_rate>
         <plugin filename="libgazebo_ros_imu_sensor.so" name="imu_plugin">
-          <!-- <robotNamespace>${robot_ns}</robotNamespace> -->
           <topicName>zed2/imu/data</topicName>
           <frameName>zed2_imu_link</frameName>
