Commit message: Revert to gazebo plugin for robot control, update README

File: parc_robot_description/urdf/enclosure.xacro (robot description, xacro)
@@ -12,7 +12,7 @@
         <origin xyz="0 0 0" rpy="0 0 0" />
         <geometry>
-          <!-- <mesh filename="package://parc_robot/meshes/enclosure.dae" scale="0.001 0.001 0.001" /> -->
+          <mesh filename="package://parc_robot_description/meshes/enclosure.dae" scale="0.001 0.001 0.001" />
           <!-- <mesh filename="package://parc_robot/meshes/enclosure_with_overhang.stl" scale="0.001 0.001 0.001" /> -->
-          <mesh filename="package://parc_robot_description/meshes/enclosure_with_overhang.dae" scale="0.001 0.001 0.001" />
+          <!-- <mesh filename="package://parc_robot_description/meshes/enclosure_with_overhang.dae" scale="0.001 0.001 0.001" /> -->
         </geometry>
         <!-- <material name="dirty_metal">
@@ -30,7 +30,7 @@
         <origin xyz="0 0 0" rpy="0 0 0" />
         <geometry>
-          <!-- <mesh filename="package://parc_robot/meshes/enclosure.dae" scale="0.001 0.001 0.001" /> -->
+          <mesh filename="package://parc_robot_description/meshes/enclosure.dae" scale="0.001 0.001 0.001" />
           <!-- <mesh filename="package://parc_robot/meshes/enclosure_with_overhang.stl" scale="0.001 0.001 0.001" /> -->
-          <mesh filename="package://parc_robot_description/meshes/enclosure_with_overhang.dae" scale="0.001 0.001 0.001" />
+          <!-- <mesh filename="package://parc_robot_description/meshes/enclosure_with_overhang.dae" scale="0.001 0.001 0.001" /> -->
         </geometry>
       </collision>

File: parc_robot_description/urdf/parc_robot.xacro (robot description, xacro)
@@ -2,5 +2,4 @@
 <robot name="parc_robot_v2" xmlns:xacro="http://ros.org/wiki/xacro">
   <xacro:arg name="robot_namespace" default="/" />
-  <xacro:arg name="urdf_extras" default="empty.urdf" />
   <xacro:include filename="$(find parc_robot_description)/urdf/scout_wheel_type1.xacro" />
   <xacro:include filename="$(find parc_robot_description)/urdf/scout_wheel_type2.xacro" />
@@ -37,10 +36,13 @@
       </collision>
   </link>
+  <link name="base_footprint"/>
+  <joint name="base_footprint_joint" type="fixed">
+      <origin xyz="0 0 ${wheel_vertical_offset - wheel_radius}" rpy="0 0 0" />
+      <parent link="base_link" />
+      <child link="base_footprint" />
+  </joint>
   <link name="inertial_link">
       <inertial>
           <mass value="40" />
-          <!-- <mass value="50" /> -->
-          <!-- <origin xyz="-0.00065 -0.085 0.062" />
-          <inertia ixx="0.6022" ixy="-0.02364" ixz="-0.1197" iyy="1.7386" iyz="-0.001544" izz="2.0296" /> -->
           <origin xyz="0.0 0.0 0.0" />
           <inertia ixx="2.288641" ixy="0" ixz="0" iyy="5.103976" iyz="0" izz="3.431465" />
@@ -67,4 +69,23 @@
       <origin xyz="${-wheelbase/2} ${-track/2} ${wheel_vertical_offset}" rpy="3.142 0 0" />
   </xacro:scout_wheel_type2>
+  <!-- <gazebo reference="front_right_wheel"> -->
+  <!--   <mu1 value="0.5"/> -->
+  <!--   <mu2 value="0.5"/> -->
+  <!-- </gazebo> -->
+  <!---->
+  <!-- <gazebo reference="rear_right_wheel"> -->
+  <!--   <mu1 value="0.5"/> -->
+  <!--   <mu2 value="0.5"/> -->
+  <!-- </gazebo> -->
+  <!---->
+  <!-- <gazebo reference="front_left_wheel"> -->
+  <!--   <mu1 value="0.5"/> -->
+  <!--   <mu2 value="0.5"/> -->
+  <!-- </gazebo> -->
+  <!---->
+  <!-- <gazebo reference="rear_left_wheel"> -->
+  <!--   <mu1 value="0.5"/> -->
+  <!--   <mu2 value="0.5"/> -->
+  <!-- </gazebo> -->
   <!-- Sensor definitions -->
   <xacro:include filename="$(find parc_robot_description)/urdf/sensors.xacro" />

File: parc_robot_description/urdf/parc_robot_gazebo.xacro (robot description, xacro)
@@ -1,41 +1,4 @@
 <?xml version="1.0"?>
 <robot xmlns:xacro="http://ros.org/wiki/xacro">
-  <ros2_control name='GazeboSystem' type='system'>
-    <hardware>
-      <plugin>gazebo_ros2_control/GazeboSystem</plugin>
-    </hardware>
-    <joint name='front_left_wheel'>
-      <command_interface name='velocity'>
-        <param name='min'>-10</param>
-        <param name='max'>10</param>
-      </command_interface>
-      <state_interface name='velocity'/>
-      <state_interface name='position'/>
-    </joint>
-    <joint name='front_right_wheel'>
-      <command_interface name='velocity'>
-        <param name='min'>-10</param>
-        <param name='max'>10</param>
-      </command_interface>
-      <state_interface name='velocity'/>
-      <state_interface name='position'/>
-    </joint>
-    <joint name='rear_left_wheel'>
-      <command_interface name='velocity'>
-        <param name='min'>-10</param>
-        <param name='max'>10</param>
-      </command_interface>
-      <state_interface name='velocity'/>
-      <state_interface name='position'/>
-    </joint>
-    <joint name='rear_right_wheel'>
-      <command_interface name='velocity'>
-        <param name='min'>-10</param>
-        <param name='max'>10</param>
-      </command_interface>
-      <state_interface name='velocity'/>
-      <state_interface name='position'/>
-    </joint>
-  </ros2_control>
   <gazebo>
     <mu1 value="1.0"/>
@@ -48,7 +11,21 @@
   </gazebo>
   <gazebo>
-    <plugin name='gazebo_ros2_control' filename='libgazebo_ros2_control.so'>
-      <parameters>$(find parc_robot_bringup)/config/controllers.yaml</parameters>
-      <parameters>$(find parc_robot_bringup)/config/gazebo_ros2_ctl_use_sim.yaml</parameters>
+    <plugin name="parc_robot_skid_steer_drive" filename="libgazebo_ros_diff_drive.so">
+      <!-- Wheel information -->
+      <num_wheel_pairs>2</num_wheel_pairs>
+      <left_joint>front_left_wheel</left_joint>
+      <left_joint>rear_left_wheel</left_joint>
+      <right_joint>front_right_wheel</right_joint>
+      <right_joint>rear_right_wheel</right_joint>
+      <wheel_separation>0.498</wheel_separation>
+      <wheel_diameter>0.370</wheel_diameter>
+      <max_wheel_torque>1000</max_wheel_torque>
+      <max_wheel_acceleration>2</max_wheel_acceleration>
+      <!-- Output -->
+      <odometry_frame>odom</odometry_frame>
+      <robot_base_frame>base_link</robot_base_frame>
+      <publish_odom>true</publish_odom>
+      <publish_odom_tf>true</publish_odom_tf>
+      <publish_wheel_tf>true</publish_wheel_tf>
     </plugin>
   </gazebo>

File: parc_robot_description/urdf/sensors.xacro (robot description, xacro)
@@ -3,5 +3,5 @@
   <!-- Includes -->
   <xacro:include filename="$(find parc_robot_description)/urdf/ydlidar.xacro" />
-  <xacro:include filename="$(find parc_robot_description)/urdf/zed2.xacro" />
+  <!-- <xacro:include filename="$(find parc_robot_description)/urdf/zed2.xacro" /> -->
   <xacro:include filename="$(find parc_robot_description)/urdf/gps.xacro" />
   <xacro:include filename="$(find parc_robot_description)/urdf/side_cameras.xacro" />
@@ -11,7 +11,7 @@
   </xacro:ydlidar_sensor>
   <!-- zed2 camera -->
-  <xacro:zed2 parent="base_link">
-    <origin xyz="0.36 0 0.11" rpy="0 0 0"/>
-  </xacro:zed2>
+  <!-- <xacro:zed2 parent="base_link"> -->
+  <!--   <origin xyz="0.36 0 0.11" rpy="0 0 0"/> -->
+  <!-- </xacro:zed2> -->
   <!-- gps -->
   <xacro:gps_sensor parent="base_link">
@@ -20,9 +20,9 @@
   <!-- left_side_camera -->
   <xacro:left_side_camera parent="base_link">
-    <origin xyz="0 0.55 0.635" rpy="0 1.5708 1.571428571"/>
+    <origin xyz="0.0 0.242 0.635" rpy="0 0 ${pi/2}"/>
   </xacro:left_side_camera>
     <!-- right_side_camera -->
   <xacro:right_side_camera parent="base_link">
-    <origin xyz="0 -0.55 0.635" rpy="0 1.5708 1.571428571"/>
+    <origin xyz="0.0 -0.241 0.635" rpy="0 0 -${pi/2}"/>
   </xacro:right_side_camera>
 </robot>

File: parc_robot_description/urdf/side_cameras.xacro (robot description, xacro)
@@ -14,5 +14,4 @@
       </inertial>
       <visual>
-        <origin xyz="0.0 0.015 0.0" rpy="0 -${pi/2} 0"/>
         <geometry>
           <mesh filename="package://parc_robot_description/meshes/ZED2.dae"/>
@@ -20,5 +19,4 @@
       </visual>
       <collision>
-        <origin xyz="0.0 0.015 0.0" rpy="0 0 0"/>
         <geometry>
           <mesh filename="package://parc_robot_description/meshes/ZED2.dae"/>
@@ -31,4 +29,5 @@
       <parent link="${parent}" />
       <child link="left_camera" />
+      <origin xyz="0 0 0" rpy="0 ${pi/2} 0"/>
     </joint>
     <!-- Left Camera Gazebo -->
@@ -90,5 +89,4 @@
       </inertial>
       <visual>
-        <origin xyz="0.0 0.015 0.0" rpy="0 ${pi/2} 0"/>
         <geometry>
           <mesh filename="package://parc_robot_description/meshes/ZED2.dae"/>
@@ -96,5 +94,4 @@
       </visual>
       <collision>
-        <origin xyz="0.0 0.015 0.0" rpy="0 0 0"/>
         <geometry>
           <mesh filename="package://parc_robot_description/meshes/ZED2.dae"/>

File: parc_robot_description/urdf/ydlidar.xacro (robot description, xacro)
@@ -68,7 +68,10 @@
           </noise>
         </ray>
-        <plugin name="gazebo_ros_${name}_controller" filename="libgazebo_ros_laser.so">
-          <topicName>/scan</topicName>
-          <frameName>${name}_link</frameName>
+        <plugin name="gazebo_ros_${name}_controller" filename="libgazebo_ros_ray_sensor.so">
+          <ros>
+              <argument>~/out:=scan</argument>
+          </ros>
+          <output_type>sensor_msgs/LaserScan</output_type>
+          <frame_name>${name}_link</frame_name>
         </plugin>
       </sensor>
