Commit message: Fix ros2_control integration and PARC robot drift, add parc_robot_teleop package

File: parc_robot_description/urdf/parc_robot_gazebo.xacro (robot description, xacro)
@@ -1,48 +1,47 @@
 <?xml version="1.0"?>
 <robot xmlns:xacro="http://ros.org/wiki/xacro">
- <!-- <ros2_control name='GazeboSystem' type='system'> -->
- <!--    <hardware> -->
- <!--      <plugin>gazebo_ros2_control/GazeboSystem</plugin> -->
- <!--    </hardware> -->
- <!--    <joint name='front_left_wheel'> -->
- <!--      <command_interface name='velocity'> -->
- <!--        <param name='min'>-10</param> -->
- <!--        <param name='max'>10</param> -->
- <!--      </command_interface> -->
- <!--      <state_interface name='velocity'/> -->
- <!--      <state_interface name='position'/> -->
- <!--    </joint> -->
- <!--    <joint name='front_right_wheel'> -->
- <!--      <command_interface name='velocity'> -->
- <!--        <param name='min'>-10</param> -->
- <!--        <param name='max'>10</param> -->
- <!--      </command_interface> -->
- <!--      <state_interface name='velocity'/> -->
- <!--      <state_interface name='position'/> -->
- <!--    </joint> -->
- <!--    <joint name='rear_left_wheel'> -->
- <!--      <command_interface name='velocity'> -->
- <!--        <param name='min'>-10</param> -->
- <!--        <param name='max'>10</param> -->
- <!--      </command_interface> -->
- <!--      <state_interface name='velocity'/> -->
- <!--      <state_interface name='position'/> -->
- <!--    </joint> -->
- <!--    <joint name='rear_right_wheel'> -->
- <!--      <command_interface name='velocity'> -->
- <!--        <param name='min'>-10</param> -->
- <!--        <param name='max'>10</param> -->
- <!--      </command_interface> -->
- <!--      <state_interface name='velocity'/> -->
- <!--      <state_interface name='position'/> -->
- <!--    </joint> -->
- <!--  </ros2_control> -->
- <!---->
- <!--  <gazebo> -->
- <!--    <plugin name='gazebo_ros2_control' filename='libgazebo_ros2_control.so'> -->
- <!--      <parameters>$(find parc_robot_bringup)/config/controllers.yaml</parameters> -->
- <!--      <parameters>$(find parc_robot_bringup)/config/gazebo_ros2_ctl_use_sim.yaml</parameters> -->
- <!--    </plugin> -->
- <!--  </gazebo> -->
+ <ros2_control name='GazeboSystem' type='system'>
+    <hardware>
+      <plugin>gazebo_ros2_control/GazeboSystem</plugin>
+    </hardware>
+    <joint name='front_left_wheel'>
+      <command_interface name='velocity'>
+        <param name='min'>-10</param>
+        <param name='max'>10</param>
+      </command_interface>
+      <state_interface name='velocity'/>
+      <state_interface name='position'/>
+    </joint>
+    <joint name='front_right_wheel'>
+      <command_interface name='velocity'>
+        <param name='min'>-10</param>
+        <param name='max'>10</param>
+      </command_interface>
+      <state_interface name='velocity'/>
+      <state_interface name='position'/>
+    </joint>
+    <joint name='rear_left_wheel'>
+      <command_interface name='velocity'>
+        <param name='min'>-10</param>
+        <param name='max'>10</param>
+      </command_interface>
+      <state_interface name='velocity'/>
+      <state_interface name='position'/>
+    </joint>
+    <joint name='rear_right_wheel'>
+      <command_interface name='velocity'>
+        <param name='min'>-10</param>
+        <param name='max'>10</param>
+      </command_interface>
+      <state_interface name='velocity'/>
+      <state_interface name='position'/>
+    </joint>
+  </ros2_control>
+  <gazebo>
+    <plugin name='gazebo_ros2_control' filename='libgazebo_ros2_control.so'>
+      <parameters>$(find parc_robot_bringup)/config/controllers.yaml</parameters>
+      <parameters>$(find parc_robot_bringup)/config/gazebo_ros2_ctl_use_sim.yaml</parameters>
+    </plugin>
+  </gazebo>
   <!-- <gazebo> -->
   <!--   <mu1 value="1.0"/> -->
@@ -54,57 +53,35 @@
   <!--   <maxContacts value="64"/> -->
   <!-- </gazebo> -->
-    <gazebo reference="front_left_wheel">
-        <mu1>0.9</mu1>
-        <mu2>0.7</mu2>
-        <kp>1000000000.0</kp>
-        <kd>0.0</kd>
-        <minDepth>0.001</minDepth>
-        <fdir1>1 0 0</fdir1>
-    </gazebo>
-    <gazebo reference="front_right_wheel">
-        <mu1>0.9</mu1>
-        <mu2>0.7</mu2>
-        <kp>1000000000.0</kp>
-        <kd>0.0</kd>
-        <minDepth>0.001</minDepth>
-        <fdir1>1 0 0</fdir1>
-    </gazebo>
-    <gazebo reference="rear_left_wheel">
-        <mu1>0.9</mu1>
-        <mu2>0.7</mu2>
-        <kp>1000000000.0</kp>
-        <kd>0.0</kd>
-        <minDepth>0.001</minDepth>
-        <fdir1>1 0 0</fdir1>
-    </gazebo>
-    <gazebo reference="rear_right_wheel">
-        <mu1>0.9</mu1>
-        <mu2>0.7</mu2>
-        <kp>1000000000.0</kp>
-        <kd>0.0</kd>
-        <minDepth>0.001</minDepth>
-        <fdir1>1 0 0</fdir1>
-    </gazebo>
-  <gazebo>
-    <plugin name="parc_robot_skid_steer_drive" filename="libgazebo_ros_diff_drive.so">
-      <!-- Wheel information -->
-      <num_wheel_pairs>2</num_wheel_pairs>
-      <left_joint>front_left_wheel</left_joint>
-      <left_joint>rear_left_wheel</left_joint>
-      <right_joint>front_right_wheel</right_joint>
-      <right_joint>rear_right_wheel</right_joint>
-      <wheel_separation>0.498</wheel_separation>
-      <wheel_diameter>0.370</wheel_diameter>
-      <max_wheel_torque>40</max_wheel_torque>
-      <!-- <max_wheel_acceleration>2</max_wheel_acceleration> -->
-      <max_wheel_acceleration>0.8</max_wheel_acceleration>
-      <!-- Output -->
-      <odometry_frame>odom</odometry_frame>
-      <!-- <robot_base_frame>base_link</robot_base_frame> -->
-      <robot_base_frame>base_footprint</robot_base_frame>
-      <publish_odom>true</publish_odom>
-      <publish_odom_tf>true</publish_odom_tf>
-      <publish_wheel_tf>true</publish_wheel_tf>
-    </plugin>
+  <gazebo reference="front_left_wheel">
+      <mu1>0.9</mu1>
+      <mu2>0.7</mu2>
+      <kp>1000000000.0</kp>
+      <kd>0.0</kd>
+      <minDepth>0.001</minDepth>
+      <fdir1>1 0 0</fdir1>
+  </gazebo>
+  <gazebo reference="front_right_wheel">
+      <mu1>0.9</mu1>
+      <mu2>0.7</mu2>
+      <kp>1000000000.0</kp>
+      <kd>0.0</kd>
+      <minDepth>0.001</minDepth>
+      <fdir1>1 0 0</fdir1>
+  </gazebo>
+  <gazebo reference="rear_left_wheel">
+      <mu1>0.9</mu1>
+      <mu2>0.7</mu2>
+      <kp>1000000000.0</kp>
+      <kd>0.0</kd>
+      <minDepth>0.001</minDepth>
+      <fdir1>1 0 0</fdir1>
+  </gazebo>
+  <gazebo reference="rear_right_wheel">
+      <mu1>0.9</mu1>
+      <mu2>0.7</mu2>
+      <kp>1000000000.0</kp>
+      <kd>0.0</kd>
+      <minDepth>0.001</minDepth>
+      <fdir1>1 0 0</fdir1>
   </gazebo>
 </robot>

File: parc_robot_description/urdf/scout_wheel_type1.xacro (robot description, xacro)
@@ -29,6 +29,5 @@
                 <mass value="3" />
                 <origin xyz="0 0 0" />
-                <inertia ixx="0.02467" ixy="0" ixz="0" iyy="0.04411" iyz="0" izz="0.02467" />
-                <!-- <inertia ixx="0.7171" ixy="0" ixz="0" iyy="0.1361" iyz="0" izz="0.7171" /> -->
+                <inertia ixx="0.7171" ixy="0" ixz="0" iyy="0.1361" iyz="0" izz="0.7171" />
             </inertial>
             <visual>

File: parc_robot_description/urdf/scout_wheel_type2.xacro (robot description, xacro)
@@ -29,6 +29,5 @@
                 <mass value="3" />
                 <origin xyz="0 0 0" />
-                <inertia ixx="0.02467" ixy="0" ixz="0" iyy="0.04411" iyz="0" izz="0.02467" />
-                <!-- <inertia ixx="0.7171" ixy="0" ixz="0" iyy="0.1361" iyz="0" izz="0.7171" /> -->
+                <inertia ixx="0.7171" ixy="0" ixz="0" iyy="0.1361" iyz="0" izz="0.7171" />
             </inertial>
             <visual>

File: parc_robot_description/urdf/sensors.xacro (robot description, xacro)
@@ -3,5 +3,5 @@
   <!-- Includes -->
   <xacro:include filename="$(find parc_robot_description)/urdf/ydlidar.xacro" />
-  <!-- <xacro:include filename="$(find parc_robot_description)/urdf/zed2.xacro" /> -->
+  <xacro:include filename="$(find parc_robot_description)/urdf/zed2.xacro" />
   <xacro:include filename="$(find parc_robot_description)/urdf/gps.xacro" />
   <xacro:include filename="$(find parc_robot_description)/urdf/side_cameras.xacro" />
@@ -11,7 +11,7 @@
   </xacro:ydlidar_sensor>
   <!-- zed2 camera -->
-  <!-- <xacro:zed2 parent="base_link"> -->
-  <!--   <origin xyz="0.36 0 0.11" rpy="0 0 0"/> -->
-  <!-- </xacro:zed2> -->
+  <xacro:zed2 parent="base_link">
+    <origin xyz="0.36 0 0.11" rpy="0 0 0"/>
+  </xacro:zed2>
   <!-- gps -->
   <xacro:gps_sensor parent="base_link">

File: parc_robot_description/urdf/zed2.xacro (robot description, xacro)
@@ -81,4 +81,10 @@
     </joint>
     <link name="zed2_temp_right_link" />
+    <joint name="zed2_imu_joint" type="fixed">
+      <parent link="zed2_camera_center"/>
+      <child link="zed2_imu_link"/>
+      <origin xyz="0 0 0" rpy="0 0 0" />
+    </joint>
+    <link name="zed2_imu_link" />
     <gazebo reference="zed2_camera_center">
       <sensor type="camera" name="zed2_center_camera">
@@ -183,17 +189,21 @@
             <width>1280</width>
             <height>720</height>
-            <format>R8G8B8</format>
-          </image>
-          <clip>
-            <near>0.02</near>
-            <far>300</far>
-          </clip>
-          <noise>
-            <type>gaussian</type>
-            <mean>0.0</mean>
-            <stddev>0.007</stddev>
-          </noise>
-        </camera>
-        <plugin name="zed2_leftd_camera_controller" filename="libgazebo_ros_openni_kinect.so">
+            <format>B8G8R8</format>
+            <!-- <format>R8G8B8</format> -->
+          </image>
+          <clip>
+            <near>0.02</near>
+            <far>300</far>
+          </clip>
+          <noise>
+            <type>gaussian</type>
+            <mean>0.0</mean>
+            <stddev>0.007</stddev>
+          </noise>
+        </camera>
+        <plugin name="zed2_leftd_camera_controller" filename="libgazebo_ros_camera.so">
+          <frame_name>zed2_left_camera_optical_frame</frame_name>
+          <!-- <min_depth>0.1</min_depth> -->
+          <!-- <max_depth>100</max_depth> -->
           <cameraName>zed2</cameraName>
           <imageTopicName>left/image_rect_color</imageTopicName>
@@ -204,5 +214,4 @@
           <pointCloudCutoff>0.3</pointCloudCutoff>
           <pointCloudCutoffMax>20.0</pointCloudCutoffMax>
-          <frameName>zed2_left_camera_optical_frame</frameName>
           <baseline>0.12</baseline>
           <CxPrime>658.8206787109375</CxPrime>

Commit message: Fix task2 navigation with Gazebo

File: parc_robot_description/urdf/parc_robot_gazebo.xacro (robot description, xacro)
@@ -37,4 +37,36 @@
       <state_interface name='position'/>
     </joint>
+    <transmission name="front_right_wheel_transmission">
+      <plugin>transmission_interface/SimpleTransmission</plugin>
+        <actuator name="front_right_wheel_motor" role="front_right_wheel_motor"/>
+        <joint name="front_right_wheel" role="front_right_wheel">
+          <mechanical_reduction>1.0</mechanical_reduction>
+          <offset>0.0</offset>
+        </joint>
+    </transmission>
+    <transmission name="rear_right_wheel_transmission">
+      <plugin>transmission_interface/SimpleTransmission</plugin>
+        <actuator name="rear_right_wheel_motor" role="rear_right_wheel_motor"/>
+        <joint name="rear_right_wheel" role="rear_right_wheel">
+          <mechanical_reduction>1.0</mechanical_reduction>
+          <offset>0.0</offset>
+        </joint>
+    </transmission>
+    <transmission name="front_left_wheel_transmission">
+      <plugin>transmission_interface/SimpleTransmission</plugin>
+        <actuator name="front_left_wheel_motor" role="front_left_wheel_motor"/>
+        <joint name="front_left_wheel" role="front_left_wheel">
+          <mechanical_reduction>1.0</mechanical_reduction>
+          <offset>0.0</offset>
+        </joint>
+    </transmission>
+    <transmission name="rear_left_wheel_transmission">
+      <plugin>transmission_interface/SimpleTransmission</plugin>
+        <actuator name="rear_left_wheel_motor" role="rear_left_wheel_motor"/>
+        <joint name="rear_left_wheel" role="rear_left_wheel">
+          <mechanical_reduction>1.0</mechanical_reduction>
+          <offset>0.0</offset>
+        </joint>
+    </transmission>
   </ros2_control>
   <gazebo>
@@ -44,35 +76,47 @@
     </plugin>
   </gazebo>
-  <gazebo reference="front_left_wheel">
-      <mu1>0.9</mu1>
-      <mu2>0.7</mu2>
-      <kp>1000000000.0</kp>
-      <kd>0.0</kd>
-      <minDepth>0.001</minDepth>
-      <fdir1>1 0 0</fdir1>
-  </gazebo>
-  <gazebo reference="front_right_wheel">
-      <mu1>0.9</mu1>
-      <mu2>0.7</mu2>
-      <kp>1000000000.0</kp>
-      <kd>0.0</kd>
-      <minDepth>0.001</minDepth>
-      <fdir1>1 0 0</fdir1>
-  </gazebo>
-  <gazebo reference="rear_left_wheel">
-      <mu1>0.9</mu1>
-      <mu2>0.7</mu2>
-      <kp>1000000000.0</kp>
-      <kd>0.0</kd>
-      <minDepth>0.001</minDepth>
-      <fdir1>1 0 0</fdir1>
-  </gazebo>
-  <gazebo reference="rear_right_wheel">
-      <mu1>0.9</mu1>
-      <mu2>0.7</mu2>
-      <kp>1000000000.0</kp>
-      <kd>0.0</kd>
-      <minDepth>0.001</minDepth>
-      <fdir1>1 0 0</fdir1>
-  </gazebo>
+  <!-- <gazebo> -->
+  <!--   <mu1 value="1.0"/> -->
+  <!--   <mu2 value="0.9"/> -->
+  <!--   <kp value="10000000.0" /> -->
+  <!--   <kd value="1.0" /> -->
+  <!--   <fdir1 value="1 0 0"/> -->
+  <!--   <minDepth value="0.001" /> -->
+  <!--   <maxContacts value="64"/> -->
+  <!-- </gazebo> -->
+  <!-- <gazebo reference="front_left_wheel"> -->
+  <!--     <mu1>0.9</mu1> -->
+  <!--     <mu2>0.7</mu2> -->
+  <!--     <kp>1000000000.0</kp> -->
+  <!--     <kd>0.0</kd> -->
+  <!--     <minDepth>0.001</minDepth> -->
+  <!--     <fdir1>1 0 0</fdir1> -->
+  <!-- </gazebo> -->
+  <!---->
+  <!-- <gazebo reference="front_right_wheel"> -->
+  <!--     <mu1>0.9</mu1> -->
+  <!--     <mu2>0.7</mu2> -->
+  <!--     <kp>1000000000.0</kp> -->
+  <!--     <kd>0.0</kd> -->
+  <!--     <minDepth>0.001</minDepth> -->
+  <!--     <fdir1>1 0 0</fdir1> -->
+  <!-- </gazebo> -->
+  <!---->
+  <!-- <gazebo reference="rear_left_wheel"> -->
+  <!--     <mu1>0.9</mu1> -->
+  <!--     <mu2>0.7</mu2> -->
+  <!--     <kp>1000000000.0</kp> -->
+  <!--     <kd>0.0</kd> -->
+  <!--     <minDepth>0.001</minDepth> -->
+  <!--     <fdir1>1 0 0</fdir1> -->
+  <!-- </gazebo> -->
+  <!---->
+  <!-- <gazebo reference="rear_right_wheel"> -->
+  <!--     <mu1>0.9</mu1> -->
+  <!--     <mu2>0.7</mu2> -->
+  <!--     <kp>1000000000.0</kp> -->
+  <!--     <kd>0.0</kd> -->
+  <!--     <minDepth>0.001</minDepth> -->
+  <!--     <fdir1>1 0 0</fdir1> -->
+  <!-- </gazebo> -->
 </robot>
