Commit message: Update world, robot and goal locations for task 1

File: parc_robot_description/urdf/gps.xacro (robot description, xacro)
@@ -18,5 +18,4 @@
         <always_on>true</always_on>
         <update_rate>4.0</update_rate>
-        <pose>0 0 0 0 0 0</pose>
         <gps>
           <position_sensing>
@@ -24,5 +23,5 @@
               <noise type="gaussian">
                 <mean>0.0</mean>
-                <stddev>0.01</stddev>
+                <stddev>0.001</stddev>
               </noise>
             </horizontal>
@@ -30,5 +29,5 @@
               <noise type="gaussian">
                 <mean>0.0</mean>
-                <stddev>0.01</stddev>
+                <stddev>0.001</stddev>
               </noise>
             </vertical>

File: parc_robot_description/urdf/parc_robot.xacro (robot description, xacro)
@@ -1,5 +1,4 @@
 <?xml version="1.0"?>
 <robot name="parc_robot_v2" xmlns:xacro="http://ros.org/wiki/xacro">
-  <xacro:arg name="robot_namespace" default="/" />
   <xacro:include filename="$(find parc_robot_description)/urdf/scout_wheel_type1.xacro" />
   <xacro:include filename="$(find parc_robot_description)/urdf/scout_wheel_type2.xacro" />
@@ -38,7 +37,7 @@
   <link name="base_footprint"/>
   <joint name="base_footprint_joint" type="fixed">
-      <origin xyz="0 0 ${wheel_vertical_offset - wheel_radius}" rpy="0 0 0" />
-      <parent link="base_link" />
-      <child link="base_footprint" />
+      <origin xyz="0 0 ${wheel_radius - wheel_vertical_offset}" rpy="0 0 0" />
+      <parent link="base_footprint" />
+      <child link="base_link" />
   </joint>
   <link name="inertial_link">
@@ -69,23 +68,4 @@
       <origin xyz="${-wheelbase/2} ${-track/2} ${wheel_vertical_offset}" rpy="3.142 0 0" />
   </xacro:scout_wheel_type2>
-  <!-- <gazebo reference="front_right_wheel"> -->
-  <!--   <mu1 value="0.5"/> -->
-  <!--   <mu2 value="0.5"/> -->
-  <!-- </gazebo> -->
-  <!---->
-  <!-- <gazebo reference="rear_right_wheel"> -->
-  <!--   <mu1 value="0.5"/> -->
-  <!--   <mu2 value="0.5"/> -->
-  <!-- </gazebo> -->
-  <!---->
-  <!-- <gazebo reference="front_left_wheel"> -->
-  <!--   <mu1 value="0.5"/> -->
-  <!--   <mu2 value="0.5"/> -->
-  <!-- </gazebo> -->
-  <!---->
-  <!-- <gazebo reference="rear_left_wheel"> -->
-  <!--   <mu1 value="0.5"/> -->
-  <!--   <mu2 value="0.5"/> -->
-  <!-- </gazebo> -->
   <!-- Sensor definitions -->
   <xacro:include filename="$(find parc_robot_description)/urdf/sensors.xacro" />

File: parc_robot_description/urdf/parc_robot_gazebo.xacro (robot description, xacro)
@@ -1,13 +1,89 @@
 <?xml version="1.0"?>
 <robot xmlns:xacro="http://ros.org/wiki/xacro">
-  <gazebo>
-    <mu1 value="1.0"/>
-    <mu2 value="0.9"/>
-    <kp value="10000000.0" />
-    <kd value="1.0" />
-    <fdir1 value="1 0 0"/>
-    <minDepth value="0.001" />
-    <maxContacts value="64"/>
-  </gazebo>
+ <!-- <ros2_control name='GazeboSystem' type='system'> -->
+ <!--    <hardware> -->
+ <!--      <plugin>gazebo_ros2_control/GazeboSystem</plugin> -->
+ <!--    </hardware> -->
+ <!--    <joint name='front_left_wheel'> -->
+ <!--      <command_interface name='velocity'> -->
+ <!--        <param name='min'>-10</param> -->
+ <!--        <param name='max'>10</param> -->
+ <!--      </command_interface> -->
+ <!--      <state_interface name='velocity'/> -->
+ <!--      <state_interface name='position'/> -->
+ <!--    </joint> -->
+ <!--    <joint name='front_right_wheel'> -->
+ <!--      <command_interface name='velocity'> -->
+ <!--        <param name='min'>-10</param> -->
+ <!--        <param name='max'>10</param> -->
+ <!--      </command_interface> -->
+ <!--      <state_interface name='velocity'/> -->
+ <!--      <state_interface name='position'/> -->
+ <!--    </joint> -->
+ <!--    <joint name='rear_left_wheel'> -->
+ <!--      <command_interface name='velocity'> -->
+ <!--        <param name='min'>-10</param> -->
+ <!--        <param name='max'>10</param> -->
+ <!--      </command_interface> -->
+ <!--      <state_interface name='velocity'/> -->
+ <!--      <state_interface name='position'/> -->
+ <!--    </joint> -->
+ <!--    <joint name='rear_right_wheel'> -->
+ <!--      <command_interface name='velocity'> -->
+ <!--        <param name='min'>-10</param> -->
+ <!--        <param name='max'>10</param> -->
+ <!--      </command_interface> -->
+ <!--      <state_interface name='velocity'/> -->
+ <!--      <state_interface name='position'/> -->
+ <!--    </joint> -->
+ <!--  </ros2_control> -->
+ <!---->
+ <!--  <gazebo> -->
+ <!--    <plugin name='gazebo_ros2_control' filename='libgazebo_ros2_control.so'> -->
+ <!--      <parameters>$(find parc_robot_bringup)/config/controllers.yaml</parameters> -->
+ <!--      <parameters>$(find parc_robot_bringup)/config/gazebo_ros2_ctl_use_sim.yaml</parameters> -->
+ <!--    </plugin> -->
+ <!--  </gazebo> -->
+  <!-- <gazebo> -->
+  <!--   <mu1 value="1.0"/> -->
+  <!--   <mu2 value="0.9"/> -->
+  <!--   <kp value="10000000.0" /> -->
+  <!--   <kd value="1.0" /> -->
+  <!--   <fdir1 value="1 0 0"/> -->
+  <!--   <minDepth value="0.001" /> -->
+  <!--   <maxContacts value="64"/> -->
+  <!-- </gazebo> -->
+    <gazebo reference="front_left_wheel">
+        <mu1>0.9</mu1>
+        <mu2>0.7</mu2>
+        <kp>1000000000.0</kp>
+        <kd>0.0</kd>
+        <minDepth>0.001</minDepth>
+        <fdir1>1 0 0</fdir1>
+    </gazebo>
+    <gazebo reference="front_right_wheel">
+        <mu1>0.9</mu1>
+        <mu2>0.7</mu2>
+        <kp>1000000000.0</kp>
+        <kd>0.0</kd>
+        <minDepth>0.001</minDepth>
+        <fdir1>1 0 0</fdir1>
+    </gazebo>
+    <gazebo reference="rear_left_wheel">
+        <mu1>0.9</mu1>
+        <mu2>0.7</mu2>
+        <kp>1000000000.0</kp>
+        <kd>0.0</kd>
+        <minDepth>0.001</minDepth>
+        <fdir1>1 0 0</fdir1>
+    </gazebo>
+    <gazebo reference="rear_right_wheel">
+        <mu1>0.9</mu1>
+        <mu2>0.7</mu2>
+        <kp>1000000000.0</kp>
+        <kd>0.0</kd>
+        <minDepth>0.001</minDepth>
+        <fdir1>1 0 0</fdir1>
+    </gazebo>
   <gazebo>
     <plugin name="parc_robot_skid_steer_drive" filename="libgazebo_ros_diff_drive.so">
@@ -20,9 +96,11 @@
       <wheel_separation>0.498</wheel_separation>
       <wheel_diameter>0.370</wheel_diameter>
-      <max_wheel_torque>1000</max_wheel_torque>
-      <max_wheel_acceleration>2</max_wheel_acceleration>
+      <max_wheel_torque>40</max_wheel_torque>
+      <!-- <max_wheel_acceleration>2</max_wheel_acceleration> -->
+      <max_wheel_acceleration>0.8</max_wheel_acceleration>
       <!-- Output -->
       <odometry_frame>odom</odometry_frame>
-      <robot_base_frame>base_link</robot_base_frame>
+      <!-- <robot_base_frame>base_link</robot_base_frame> -->
+      <robot_base_frame>base_footprint</robot_base_frame>
       <publish_odom>true</publish_odom>
       <publish_odom_tf>true</publish_odom_tf>

File: parc_robot_description/urdf/scout_wheel_type1.xacro (robot description, xacro)
@@ -29,5 +29,6 @@
                 <mass value="3" />
                 <origin xyz="0 0 0" />
-                <inertia ixx="0.7171" ixy="0" ixz="0" iyy="0.1361" iyz="0" izz="0.7171" />
+                <inertia ixx="0.02467" ixy="0" ixz="0" iyy="0.04411" iyz="0" izz="0.02467" />
+                <!-- <inertia ixx="0.7171" ixy="0" ixz="0" iyy="0.1361" iyz="0" izz="0.7171" /> -->
             </inertial>
             <visual>

File: parc_robot_description/urdf/scout_wheel_type2.xacro (robot description, xacro)
@@ -29,5 +29,6 @@
                 <mass value="3" />
                 <origin xyz="0 0 0" />
-                <inertia ixx="0.7171" ixy="0" ixz="0" iyy="0.1361" iyz="0" izz="0.7171" />
+                <inertia ixx="0.02467" ixy="0" ixz="0" iyy="0.04411" iyz="0" izz="0.02467" />
+                <!-- <inertia ixx="0.7171" ixy="0" ixz="0" iyy="0.1361" iyz="0" izz="0.7171" /> -->
             </inertial>
             <visual>

Commit message: Add worlds for task 2

File: parc_robot_description/urdf/gps.xacro (robot description, xacro)
@@ -18,4 +18,5 @@
         <always_on>true</always_on>
         <update_rate>4.0</update_rate>
+        <!-- <pose>0 0 0 0 0 3.14</pose> -->
         <gps>
           <position_sensing>

File: parc_robot_description/urdf/parc_robot_gazebo.xacro (robot description, xacro)
@@ -73,5 +73,5 @@
     <plugin name='gazebo_ros2_control' filename='libgazebo_ros2_control.so'>
       <parameters>$(find parc_robot_bringup)/config/controllers.yaml</parameters>
-      <parameters>$(find parc_robot_bringup)/config/gazebo_ros2_ctl_use_sim.yaml</parameters>
+      <!-- <parameters>$(find parc_robot_bringup)/config/gazebo_ros2_ctl_use_sim.yaml</parameters> -->
     </plugin>
   </gazebo>

File: parc_robot_description/urdf/sensors.xacro (robot description, xacro)
@@ -16,5 +16,6 @@
   <!-- gps -->
   <xacro:gps_sensor parent="base_link">
-    <origin xyz="0 0 0.2" rpy="0 0 0"/>
+    <!-- <origin xyz="0 0 0.2" rpy="0 0 0"/> -->
+    <origin xyz="0 0 0.2" rpy="0 0 ${pi}"/>
   </xacro:gps_sensor>
   <!-- left_side_camera -->

Commit message: Fix gps use for task 1

File: parc_robot_description/urdf/gps.xacro (robot description, xacro)
@@ -18,5 +18,4 @@
         <always_on>true</always_on>
         <update_rate>4.0</update_rate>
-        <!-- <pose>0 0 0 0 0 3.14</pose> -->
         <gps>
           <position_sensing>

File: parc_robot_description/urdf/parc_robot_gazebo.xacro (robot description, xacro)
@@ -73,5 +73,5 @@
     <plugin name='gazebo_ros2_control' filename='libgazebo_ros2_control.so'>
       <parameters>$(find parc_robot_bringup)/config/controllers.yaml</parameters>
-      <!-- <parameters>$(find parc_robot_bringup)/config/gazebo_ros2_ctl_use_sim.yaml</parameters> -->
+      <parameters>$(find parc_robot_bringup)/config/gazebo_ros2_ctl_use_sim.yaml</parameters>
     </plugin>
   </gazebo>

File: parc_robot_description/urdf/sensors.xacro (robot description, xacro)
@@ -16,6 +16,5 @@
   <!-- gps -->
   <xacro:gps_sensor parent="base_link">
-    <!-- <origin xyz="0 0 0.2" rpy="0 0 0"/> -->
-    <origin xyz="0 0 0.2" rpy="0 0 ${pi}"/>
+    <origin xyz="0 0 0.2" rpy="0 0 0"/>
   </xacro:gps_sensor>
   <!-- left_side_camera -->
