Commit message: add imu sensor and remove zed2 imu

File: parc_robot_description/urdf/sensors.xacro (robot description, xacro)
@@ -6,4 +6,5 @@
   <xacro:include filename="$(find parc_robot_description)/urdf/gps.xacro" />
   <xacro:include filename="$(find parc_robot_description)/urdf/side_cameras.xacro" />
+  <xacro:include filename="$(find parc_robot_description)/urdf/imu.xacro" />
   <!-- ydlidar -->
   <xacro:ydlidar_sensor parent="base_link">
@@ -18,4 +19,8 @@
     <origin xyz="0 0 0.2" rpy="0 0 0"/>
   </xacro:gps_sensor>
+  <!-- imu -->
+  <xacro:imu_sensor parent="base_link">
+    <origin xyz="0 0 0.3" rpy="0 0 0"/>
+  </xacro:imu_sensor>
   <!-- left_side_camera -->
   <xacro:left_side_camera parent="base_link">

File: parc_robot_description/urdf/zed2.xacro (robot description, xacro)
@@ -305,19 +305,19 @@
     </gazebo>
     <!-- IMU -->
-    <gazebo reference="zed2_left_camera_frame">
+    <!-- <gazebo reference="zed2_left_camera_frame">
       <sensor type="imu" name="zed2_imu_sensor">
         <update_rate>100</update_rate>
         <plugin filename="libgazebo_ros_imu_sensor.so" name="imu_plugin">
-          <topicName>zed2/imu/data</topicName>
-          <frameName>zed2_imu_link</frameName>
-          <updateRateHZ>100.0</updateRateHZ>
-          <gaussianNoise>0.01</gaussianNoise>
-          <initialOrientationAsReference>false</initialOrientationAsReference>
-          <!-- IMU frame offset copied from an actual ZED2 camera -->
-          <xyzOffset>-0.002 -0.023 -0.002</xyzOffset>
-          <rpyOffset>0.0014025 -0.0000012 -0.0016915</rpyOffset>
-        </plugin>
-      </sensor>
-    </gazebo>
+            <topicName>imu</topicName>
+            <bodyName>imu_link</bodyName>
+            <updateRateHZ>10.0</updateRateHZ>
+            <gaussianNoise>0.0</gaussianNoise>
+            <xyzOffset>0 0 0</xyzOffset>
+            <rpyOffset>0 0 0</rpyOffset>
+            <frame_name>imu_link</frame_name>
+            <initialOrientationAsReference>false</initialOrientationAsReference>
+        </plugin>
+      </sensor> -->
+    <!-- </gazebo> -->
   </xacro:macro>
 </robot>
